File: pcb/elevator-motherboard-revA.sch (EAGLE design)
At the start: 71 parts, among them J3 MAGJACK, J4 MAGJACK, J5 MAGJACK, J6 POWER_JACK, J8 MAGJACK, Q1 NCV8403BDTRKG, Q2 MOSFET_NCH_DUAL-SO08, Q3 MOSFET_NCH_DUAL-SO08, Q4 MOSFET_NCH_DUAL-SO08, Q5 NCV8403BDTRKG, Q6 MOSFET_NCH_DUAL-SO08, Q7 NCV8403BDTRKG, Q8 NCV8403BDTRKG, Q9 NCV8403BDTRKG, U2 TPD2E001, U3 TPD2E001, U4 74HC2G125, U5 TPD2E001, U7 TPD2E001, X1 MSTBA2, X2 MSTBA2, X3 MSTBA2, X4 MSTBA2

Commit message: Done with routing
Parts:
- added C2: 0.1uF, microbuilder:CAP_CERAMIC0603
- added H1, H2, H3, H4: MOUNT-HOLE3.2, holes:MOUNT-HOLE3.2
Connections:
- net 5V: now also C2.P$2
- net GND: now also C2.P$1
Changed lines of the file:
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@@
 <part name="GND12" library="SparkFun-Aesthetics" deviceset="GND" device=""/>
 <part name="U$2" library="SparkFun-PowerSymbols" library_urn="urn:adsk.eagle:library:530" deviceset="AGND" device="" value="GND"/>
+<part name="C2" library="microbuilder" deviceset="CAP_CERAMIC" device="0603" value="0.1uF"/>
+<part name="H1" library="holes" library_urn="urn:adsk.eagle:library:237" deviceset="MOUNT-HOLE" device="3.2" package3d_urn="urn:adsk.eagle:package:14275/1"/>
+<part name="H2" library="holes" library_urn="urn:adsk.eagle:library:237" deviceset="MOUNT-HOLE" device="3.2" package3d_urn="urn:adsk.eagle:package:14275/1"/>
+<part name="H3" library="holes" library_urn="urn:adsk.eagle:library:237" deviceset="MOUNT-HOLE" device="3.2" package3d_urn="urn:adsk.eagle:package:14275/1"/>
+<part name="H4" library="holes" library_urn="urn:adsk.eagle:library:237" deviceset="MOUNT-HOLE" device="3.2" package3d_urn="urn:adsk.eagle:package:14275/1"/>
 </parts>
 <sheets>
@@
 <attribute name="VALUE" x="223.52" y="220.726" size="1.778" layer="96" align="top-center"/>
 </instance>
+<instance part="C2" gate="G$1" x="190.5" y="137.16" smashed="yes" rot="MR180">
+<attribute name="NAME" x="193.04" y="134.62" size="1.27" layer="95" font="vector" rot="MR180"/>
+<attribute name="VALUE" x="193.04" y="137.16" size="1.27" layer="96" font="vector" rot="MR180"/>
+</instance>
+<instance part="H1" gate="G$1" x="-10.16" y="185.42" smashed="yes">
+<attribute name="NAME" x="-8.128" y="186.0042" size="1.778" layer="95"/>
+<attribute name="VALUE" x="-8.128" y="182.9562" size="1.778" layer="96"/>
+</instance>
+<instance part="H2" gate="G$1" x="-10.16" y="172.72" smashed="yes">
+<attribute name="NAME" x="-8.128" y="173.3042" size="1.778" layer="95"/>
+<attribute name="VALUE" x="-8.128" y="170.2562" size="1.778" layer="96"/>
+</instance>
+<instance part="H3" gate="G$1" x="-10.16" y="160.02" smashed="yes">
+<attribute name="NAME" x="-8.128" y="160.6042" size="1.778" layer="95"/>
+<attribute name="VALUE" x="-8.128" y="157.5562" size="1.778" layer="96"/>
+</instance>
+<instance part="H4" gate="G$1" x="-10.16" y="147.32" smashed="yes">
+<attribute name="NAME" x="-8.128" y="147.9042" size="1.778" layer="95"/>
+<attribute name="VALUE" x="-8.128" y="144.8562" size="1.778" layer="96"/>
+</instance>
 </instances>
 <busses>
@@
 <wire x1="200.66" y1="127" x2="195.58" y2="127" width="0.1524" layer="91"/>
 <wire x1="195.58" y1="134.62" x2="195.58" y2="127" width="0.1524" layer="91"/>
-<wire x1="195.58" y1="127" x2="195.58" y2="109.22" width="0.1524" layer="91"/>
+<wire x1="195.58" y1="127" x2="195.58" y2="119.38" width="0.1524" layer="91"/>
+<wire x1="195.58" y1="119.38" x2="195.58" y2="109.22" width="0.1524" layer="91"/>
 <wire x1="195.58" y1="109.22" x2="228.6" y2="109.22" width="0.1524" layer="91"/>
 <junction x="195.58" y="127"/>
 <junction x="228.6" y="109.22"/>
 <wire x1="228.6" y1="142.24" x2="228.6" y2="109.22" width="0.1524" layer="91"/>
+<pinref part="C2" gate="G$1" pin="P$1"/>
+<wire x1="190.5" y1="132.08" x2="190.5" y2="119.38" width="0.1524" layer="91"/>
+<wire x1="190.5" y1="119.38" x2="195.58" y2="119.38" width="0.1524" layer="91"/>
+<junction x="195.58" y="119.38"/>
 </segment>
 <segment>
@@
 <wire x1="195.58" y1="154.94" x2="220.98" y2="154.94" width="0.1524" layer="91"/>
 <junction x="220.98" y="154.94"/>
-</segment>
-<segment>
+<pinref part="C2" gate="G$1" pin="P$2"/>
+<wire x1="195.58" y1="142.24" x2="190.5" y2="142.24" width="0.1524" layer="91"/>
+<wire x1="190.5" y1="142.24" x2="190.5" y2="139.7" width="0.1524" layer="91"/>
+<junction x="195.58" y="142.24"/>
+</segment>
+<segment>
